File: eagle/Siguino/Siguino.brd (EAGLE design)
At the start: 70.5 x 38.7 mm, 34 parts, among them J1 FTDI Basic, Q1 MOSFET P-CH 20V 5.3A SOT-23, U1 ATMEGA328P_TQFP, U2 AT30TS750ATSSOP, U3 LIS3DH, Y1 8MHz

Commit message: Updated with latest 0.5 and 1.0 changes
Parts:
- removed R8: 10k, SparkFun-Resistors:0603
- added C8: 0.1uF, SparkFun-Capacitors:0603
- added U4: BME280, BME280ComponentLibrary:BME280_LGA
- U2: value AT30TS750ATSSOP -> LIS3MDLTR; device DigiKey:21-0036K -> LIS3MDLTR:LGA12R50P4X4_200X200X100
- moved U2 4.50 mm to (26.6, 8.80), turned to 0 degrees
- moved J1 1.30 mm to (23.1, 36.0)
- moved Q1 0.32 mm to (19.9, 35.6)
Connections:
- removed net N$8: R8.2, U2.3
- new net N$11: U1.2, U2.7
- new net N$9: C8.2, U2.4
- net GND: now also C8.1, U2.12, U2.2, U2.3, U4.P$1, U4.P$5, U4.P$7; no longer U2.4, U2.5, U2.6, U2.7
- net SCL: now also U2.1, U4.P$4; no longer U2.2
- net SDA: now also U2.11, U4.P$3; no longer U2.1
- net VCC: now also U2.10, U2.5, U2.6, U2.9, U4.P$2, U4.P$6, U4.P$8; no longer R8.1, U2.8
Routing:
- net N$11: track 0.00 -> 42.9 mm, vias 0 -> 2
- net GND: track 51.2 -> 73.2 mm, vias 7 -> 33
- net N$9: track 0.00 -> 9.20 mm, vias 0 -> 2
- net MAG_POW: track 44.6 -> 49.5 mm
- net VCC: track 137.8 -> 142.1 mm, vias 11 -> 13
- net SDA: track 56.9 -> 53.6 mm, vias 4 -> 7
- net N$8: track 3.09 -> 0.00 mm
- net SCL: track 65.8 -> 67.7 mm, vias 7 -> 5
- net MOSI: track 25.7 -> 24.1 mm
- net RXI: track 12.2 -> 13.8 mm
- net TXO: track 12.5 -> 14.0 mm
- net RESET: track 64.3 -> 62.8 mm
- net DTR: track 11.6 -> 12.5 mm
- net SCK: track 17.1 -> 17.7 mm
Other:
- board text added: "A1"
- board text added: "A2"
- board text added: "A6"
- board text added: "A7"
- board text added: "AH9246-W7"
- board text added: "ATMEGA328P"
- board text added: "BME280"
- board text added: "D3"
- board text added: "D6"
- board text added: "DTR"
- board text added: "GND"
- board text added: "LIS3DH"
- board text added: "LIS3MDL"
- board text added: "MAG SENSE"
- board text added: "MISO"
- board text added: "MOSI"
- board text added: "PROANT ONBOARD 868"
- board text added: "RST"
- board text added: "RXI"
- board text added: "SCK"
- board text added: "SCL"
- board text added: "SDA"
- board text added: "SS"
- board text added: "Siguino, Rev: 1.0"
- board text added: "TXO"
- board text added: "VCC"
- board text removed: "Siguino, Rev: 0.4"

Commit message: Cleaned schematic & changed antenna path on Board
Parts:
- ANT1: device proant:ONBOARD_SMD_2400 -> Siguino:PROANT_ONBOARD_SMD_2400
- BATT1: value CR2-BATTERY-HOLDERPTH -> SPARKFUN-BATTERIES_CR2-BATTERY-HOLDERPTH; device SparkFun-Batteries:BATTERYHOLDER-CR2 -> Siguino:SPARKFUN-BATTERIES_BATTERYHOLDER-CR2
- C8: value 0.1uF -> 100nF
- HALL1: value AH9246-W7 -> TR-J_AH9246-W7; device tr-j:SC-59 -> Siguino:TR-J_SC-59
- SFM1: device WiSOL:WSSFM10 -> Siguino:WISOL_WSSFM10
- U2: value LIS3MDLTR -> LIS3MDLTR_LIS3MDLTR; device LIS3MDLTR:LGA12R50P4X4_200X200X100 -> Siguino:LIS3MDLTR_LGA12R50P4X4_200X200X100
- U3: value LIS3DH -> SPARKFUN-SENSORS_LIS3DH; device SparkFun-Sensors:LGA-16-3X3 -> Siguino:SPARKFUN-SENSORS_LGA-16-3X3
- U4: device BME280ComponentLibrary:BME280_LGA -> Siguino:BME280COMPONENTLIBRARY_BME280_LGA
- moved C6 1.40 mm to (63.8, 30.9)
- moved C7 0.91 mm to (63.3, 26.6), turned to 180 degrees
Connections:
- net A0 renamed LIGHT_SENSE
- net A3 renamed LIGHT_POWER
- net D3 renamed INT1
- net MAG_OUT renamed HALL_SENSE
- net MAG_POW renamed HALL_POWER
- net N$11 renamed MAG_INT
Routing:
- net HALL_POWER: track 49.5 -> 32.3 mm, vias 4 -> 3
- net GND: track 73.2 -> 76.5 mm
- net N$7: track 5.58 -> 3.75 mm
- net N$6: track 13.1 -> 13.6 mm
- net SCK: track 17.7 -> 17.2 mm
