File: eagle/Siguino/Siguino.sch (EAGLE design)
At the start: 35 parts, among them J1 FTDI Basic, Q1 MOSFET P-CH 20V 5.3A SOT-23, U1 ATMEGA328P_TQFP, U2 LIS3MDLTR_LIS3MDLTR, U3 SPARKFUN-SENSORS_LIS3DH, U4 BME280, Y1 8MHz

Commit message: Added new components and re-organised board, unrouted
Parts:
- added C14, C17: 0.1uF, SparkFun-Capacitors:0.1UF-0603-25V-(+80/-20%)
- added C16: 10uF, SparkFun-Capacitors:0.1UF-0603-25V-(+80/-20%)
- added C18: 10uF, SparkFun-Capacitors:10UF-0603-6.3V-20%
- added D2: RED, SparkFun-LED:LED-RED0603
- added D3: GREEN, SparkFun-LED:LED-RED0603
- added J4: 10118193-0001LF, 10118193-0001LF:10118193-0001LF
- added L1: 10uH, SparkFun-Coils:INDUCTOR-0603-33NH
- added R8, R9: 1k, SparkFun-Resistors:100KOHM-0603-1/10W-1%
- added U5: FT232RL, SparkFun-IC-Comms:FT232RLSSOP
- added U6: MAX1724EZK33+T, MAXIM:MAX1724EZK33+T
- J1: value FTDI Basic -> FTDI
Connections:
- net VBATT renamed VBAT
- new net 5V: C14.2, C16.2, J4.VUSB, R8.2, R9.2, U5.VCC
- new net CTS: J1.CTS, U5.CTS
- new net N$11: D2.A, R8.1
- new net N$12: D3.A, R9.1
- new net N$13: D2.C, U5.TXLED
- new net N$14: D3.C, U5.RXLED
- new net N$15: J4.D-, U5.USBDM
- new net N$16: J4.D+, U5.USBDP
- new net N$17: L1.2, U6.!SHDN, U6.LX
- new net V33: C18.2, U6.OUT
- new net VBAT2: C15.2, C3.2, L1.1, Q1.S, U6.BATT
- net DTR: now also U5.DTR
- net GND: now also C14.1, C16.1, C17.1, C18.1, J4.GND, U5.AGND, U5.GND18, U5.GND21, U5.GND7, U6.GND; no longer J1.CTS
- net RXI: now also U5.RXD
- net TXO: now also U5.TXD
- net VCC: now also C17.2, U5.3V3OUT; no longer C15.2, C3.2, Q1.S

Commit message: Finalised v2.0 and re-routed, gerbers created
Parts:
- added Q2: MOSFET P-CH 20V 5.3A SOT-23, SparkFun-DiscreteSemi:MOSFET_PCHSI2323DDS
- ANT1: value PROOB471 -> PROOB518
Connections:
- removed net V33: C18.2, U6.OUT
- new net 3V3FTDI: C17.2, Q2.D, U5.3V3OUT, U5.VCCIO
- net GND: now also J4.SHIELD, Q2.G
- net VBAT2: now also J1.VCC, Q2.S
- net VCC: now also C18.2, U6.OUT; no longer C17.2, J1.VCC, U5.3V3OUT
Changed lines of the file:
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@@
 <part name="GND14" library="SparkFun-PowerSymbols" deviceset="GND" device=""/>
 <part name="SUPPLY5" library="SparkFun-PowerSymbols" deviceset="VCC" device=""/>
-<part name="ANT1" library="Siguino" deviceset="PROANT_PRO-OB-512" device="ONBOARD" value="PROOB471"/>
+<part name="ANT1" library="Siguino" deviceset="PROANT_PRO-OB-512" device="ONBOARD" value="PROOB518"/>
 <part name="R6" library="SparkFun-Resistors" deviceset="10KOHM" device="-0603-1/10W-1%" value="10k"/>
 <part name="SUPPLY8" library="SparkFun-PowerSymbols" deviceset="VCC" device=""/>
@@
 <part name="L1" library="SparkFun-Coils" library_urn="urn:adsk.eagle:library:512" deviceset="INDUCTOR" device="-0603-33NH" package3d_urn="urn:adsk.eagle:package:37574/1" value="10uH"/>
 <part name="C18" library="SparkFun-Capacitors" deviceset="10UF" device="-0603-6.3V-20%" value="10uF"/>
+<part name="Q2" library="SparkFun-DiscreteSemi" deviceset="MOSFET_PCH" device="SI2323DDS" value="MOSFET P-CH 20V 5.3A SOT-23"/>
 </parts>
 <sheets>
@@
 <attribute name="NAME" x="397.256" y="93.599" size="1.778" layer="95" font="vector" rot="R180"/>
 <attribute name="VALUE" x="397.256" y="98.679" size="1.778" layer="96" font="vector" rot="R180"/>
+</instance>
+<instance part="Q2" gate="G$1" x="358.14" y="78.74" smashed="yes" rot="R180">
+<attribute name="NAME" x="353.06" y="78.74" size="1.778" layer="95" font="vector" rot="R180"/>
 </instance>
 </instances>
@@
 <wire x1="330.2" y1="53.34" x2="335.28" y2="53.34" width="0.1524" layer="91"/>
 <pinref part="GND21" gate="1" pin="GND"/>
-<wire x1="335.28" y1="53.34" x2="335.28" y2="63.5" width="0.1524" layer="91"/>
+<wire x1="335.28" y1="53.34" x2="335.28" y2="58.42" width="0.1524" layer="91"/>
+<pinref part="J4" gate="G$1" pin="SHIELD"/>
+<wire x1="335.28" y1="58.42" x2="335.28" y2="63.5" width="0.1524" layer="91"/>
+<wire x1="330.2" y1="58.42" x2="335.28" y2="58.42" width="0.1524" layer="91"/>
+<junction x="335.28" y="58.42"/>
 </segment>
 <segment>
@@
 <label x="398.78" y="88.9" size="1.27" layer="95" rot="R270" xref="yes"/>
 </segment>
+<segment>
+<pinref part="Q2" gate="G$1" pin="G"/>
+<wire x1="363.22" y1="81.28" x2="368.3" y2="81.28" width="0.1524" layer="91"/>
+<label x="368.3" y="81.28" size="1.778" layer="95"/>
+</segment>
 </net>
 <net name="VCC" class="0">
@@
 <wire x1="53.34" y1="60.96" x2="48.26" y2="60.96" width="0.1524" layer="91"/>
 <junction x="48.26" y="60.96"/>
-</segment>
-<segment>
-<pinref part="J1" gate="G$1" pin="VCC"/>
-<wire x1="15.24" y1="116.84" x2="17.78" y2="116.84" width="0.1524" layer="91"/>
-<label x="17.78" y="116.84" size="1.27" layer="95" xref="yes"/>
 </segment>
 <segment>
@@
 </segment>
 <segment>
-<pinref part="U5" gate="G$1" pin="3V3OUT"/>
-<wire x1="373.38" y1="40.64" x2="365.76" y2="40.64" width="0.1524" layer="91"/>
-<pinref part="C17" gate="G$1" pin="2"/>
-<wire x1="365.76" y1="40.64" x2="360.68" y2="40.64" width="0.1524" layer="91"/>
-<wire x1="365.76" y1="38.1" x2="365.76" y2="40.64" width="0.1524" layer="91"/>
-<junction x="365.76" y="40.64"/>
-<label x="360.68" y="40.64" size="1.27" layer="95" rot="R180" xref="yes"/>
+<pinref part="U6" gate="A" pin="OUT"/>
+<wire x1="393.7" y1="106.68" x2="398.78" y2="106.68" width="0.1524" layer="91"/>
+<pinref part="C18" gate="G$1" pin="2"/>
+<wire x1="398.78" y1="106.68" x2="398.78" y2="99.06" width="0.1524" layer="91"/>
+<wire x1="398.78" y1="106.68" x2="408.94" y2="106.68" width="0.1524" layer="91"/>
+<junction x="398.78" y="106.68"/>
+<label x="408.94" y="106.68" size="1.27" layer="95" xref="yes"/>
 </segment>
 </net>
@@
 </segment>
 </net>
-<net name="V33" class="0">
-<segment>
-<pinref part="U6" gate="A" pin="OUT"/>
-<wire x1="393.7" y1="106.68" x2="398.78" y2="106.68" width="0.1524" layer="91"/>
-<pinref part="C18" gate="G$1" pin="2"/>
-<wire x1="398.78" y1="106.68" x2="398.78" y2="99.06" width="0.1524" layer="91"/>
-<wire x1="398.78" y1="106.68" x2="408.94" y2="106.68" width="0.1524" layer="91"/>
-<junction x="398.78" y="106.68"/>
-<label x="408.94" y="106.68" size="1.27" layer="95" xref="yes"/>
-</segment>
-</net>
 <net name="N$17" class="0">
 <segment>
@@
 <wire x1="358.14" y1="121.92" x2="370.84" y2="121.92" width="0.1524" layer="91"/>
 </segment>
-</net>
+<segment>
+<pinref part="Q2" gate="G$1" pin="S"/>
+<wire x1="355.6" y1="83.82" x2="355.6" y2="88.9" width="0.1524" layer="91"/>
+<label x="355.6" y="88.9" size="1.27" layer="95" rot="R90" xref="yes"/>
+</segment>
+<segment>
+<pinref part="J1" gate="G$1" pin="VCC"/>
+<wire x1="15.24" y1="116.84" x2="17.78" y2="116.84" width="0.1524" layer="91"/>
+<label x="17.78" y="116.84" size="1.27" layer="95" xref="yes"/>
+</segment>
+</net>
+<net name="3V3FTDI" class="0">
+<segment>
+<pinref part="U5" gate="G$1" pin="3V3OUT"/>
+<wire x1="373.38" y1="40.64" x2="370.84" y2="40.64" width="0.1524" layer="91"/>
+<pinref part="C17" gate="G$1" pin="2"/>
+<wire x1="370.84" y1="40.64" x2="365.76" y2="40.64" width="0.1524" layer="91"/>
+<wire x1="365.76" y1="40.64" x2="360.68" y2="40.64" width="0.1524" layer="91"/>
+<wire x1="365.76" y1="38.1" x2="365.76" y2="40.64" width="0.1524" layer="91"/>
+<junction x="365.76" y="40.64"/>
+<label x="360.68" y="40.64" size="1.27" layer="95" rot="R180" xref="yes"/>
+<pinref part="U5" gate="G$1" pin="VCCIO"/>
+<wire x1="373.38" y1="38.1" x2="370.84" y2="38.1" width="0.1524" layer="91"/>
+<wire x1="370.84" y1="38.1" x2="370.84" y2="40.64" width="0.1524" layer="91"/>
+<junction x="370.84" y="40.64"/>
+</segment>
+<segment>
+<pinref part="Q2" gate="G$1" pin="D"/>
+<wire x1="355.6" y1="73.66" x2="355.6" y2="68.58" width="0.1524" layer="91"/>
+<label x="355.6" y="68.58" size="1.27" layer="95" rot="R270" xref="yes"/>
+</segment>
+</net>

Commit message: Fixed hatching issue on antenna pads, fixed FTDI problem
Parts:
- ANT1: device Siguino:PROANT_PRO-OB-512ONBOARD -> proant:PRO-OB-512ONBOARD
Connections:
- net CTS: no longer U5.CTS
- net GND: now also U5.CTS, U5.TEST
- net RXI: now also U5.TXD; no longer U5.RXD
- net TXO: now also U5.RXD; no longer U5.TXD
Changed lines of the file:
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@@
 <part name="GND14" library="SparkFun-PowerSymbols" deviceset="GND" device=""/>
 <part name="SUPPLY5" library="SparkFun-PowerSymbols" deviceset="VCC" device=""/>
-<part name="ANT1" library="Siguino" deviceset="PROANT_PRO-OB-512" device="ONBOARD" value="PROOB518"/>
+<part name="ANT1" library="proant" deviceset="PRO-OB-512" device="ONBOARD" value="PROOB518"/>
 <part name="R6" library="SparkFun-Resistors" deviceset="10KOHM" device="-0603-1/10W-1%" value="10k"/>
 <part name="SUPPLY8" library="SparkFun-PowerSymbols" deviceset="VCC" device=""/>
@@
 <attribute name="VALUE" x="279.4" y="84.074" size="1.778" layer="96" align="bottom-center"/>
 </instance>
-<instance part="ANT1" gate="ANT1" x="226.06" y="157.48" smashed="yes" rot="MR0">
-<attribute name="NAME" x="223.52" y="160.02" size="1.778" layer="95" rot="MR0"/>
+<instance part="ANT1" gate="ANT1" x="231.14" y="182.88" smashed="yes" rot="MR270">
+<attribute name="NAME" x="228.6" y="180.34" size="1.778" layer="95" rot="MR270"/>
 </instance>
 <instance part="R6" gate="G$1" x="53.34" y="114.3" smashed="yes" rot="R90">
@@
 <attribute name="VALUE" x="157.48" y="124.714" size="1.778" layer="96" align="bottom-center"/>
 </instance>
-<instance part="GND20" gate="1" x="233.68" y="162.56" smashed="yes" rot="R90">
-<attribute name="VALUE" x="233.934" y="162.56" size="1.778" layer="96" rot="R90" align="top-center"/>
+<instance part="GND20" gate="1" x="210.82" y="157.48" smashed="yes">
+<attribute name="VALUE" x="210.82" y="157.226" size="1.778" layer="96" align="top-center"/>
 </instance>
 <instance part="U5" gate="G$1" x="388.62" y="33.02" smashed="yes">
@@
 <pinref part="C15" gate="G$1" pin="1"/>
 <wire x1="182.88" y1="45.72" x2="182.88" y2="43.18" width="0.1524" layer="91"/>
-</segment>
-<segment>
-<pinref part="GND20" gate="1" pin="GND"/>
-<pinref part="ANT1" gate="ANT1" pin="GND"/>
 </segment>
 <segment>
@@
 <junction x="368.3" y="15.24"/>
 <pinref part="GND22" gate="1" pin="GND"/>
+<pinref part="U5" gate="G$1" pin="TEST"/>
+<wire x1="373.38" y1="25.4" x2="368.3" y2="25.4" width="0.1524" layer="91"/>
+<wire x1="368.3" y1="25.4" x2="368.3" y2="22.86" width="0.1524" layer="91"/>
+<junction x="368.3" y="22.86"/>
 </segment>
 <segment>
@@
 <wire x1="363.22" y1="81.28" x2="368.3" y2="81.28" width="0.1524" layer="91"/>
 <label x="368.3" y="81.28" size="1.778" layer="95"/>
+</segment>
+<segment>
+<pinref part="U5" gate="G$1" pin="CTS"/>
+<wire x1="403.86" y1="43.18" x2="408.94" y2="43.18" width="0.1524" layer="91"/>
+<label x="408.94" y="43.18" size="1.27" layer="95" xref="yes"/>
+</segment>
+<segment>
+<pinref part="ANT1" gate="ANT1" pin="GND"/>
+<pinref part="GND20" gate="1" pin="GND"/>
+<wire x1="210.82" y1="167.64" x2="210.82" y2="160.02" width="0.1524" layer="91"/>
 </segment>
 </net>
@@
 </segment>
 <segment>
+<pinref part="U5" gate="G$1" pin="TXD"/>
+<wire x1="403.86" y1="50.8" x2="408.94" y2="50.8" width="0.1524" layer="91"/>
+<label x="408.94" y="50.8" size="1.27" layer="95" xref="yes"/>
+</segment>
+</net>
+<net name="TXO" class="0">
+<segment>
+<pinref part="J1" gate="G$1" pin="RXI"/>
+<wire x1="15.24" y1="111.76" x2="17.78" y2="111.76" width="0.1524" layer="91"/>
+<label x="17.78" y="111.76" size="1.27" layer="95" xref="yes"/>
+</segment>
+<segment>
+<pinref part="U1" gate="U$1" pin="PD1(TXD)"/>
+<wire x1="101.6" y1="40.64" x2="104.14" y2="40.64" width="0.1524" layer="91"/>
+<label x="104.14" y="40.64" size="1.27" layer="95" xref="yes"/>
+</segment>
+<segment>
 <pinref part="U5" gate="G$1" pin="RXD"/>
 <wire x1="403.86" y1="48.26" x2="408.94" y2="48.26" width="0.1524" layer="91"/>
 <label x="408.94" y="48.26" size="1.27" layer="95" xref="yes"/>
-</segment>
-</net>
-<net name="TXO" class="0">
-<segment>
-<pinref part="J1" gate="G$1" pin="RXI"/>
-<wire x1="15.24" y1="111.76" x2="17.78" y2="111.76" width="0.1524" layer="91"/>
-<label x="17.78" y="111.76" size="1.27" layer="95" xref="yes"/>
-</segment>
-<segment>
-<pinref part="U1" gate="U$1" pin="PD1(TXD)"/>
-<wire x1="101.6" y1="40.64" x2="104.14" y2="40.64" width="0.1524" layer="91"/>
-<label x="104.14" y="40.64" size="1.27" layer="95" xref="yes"/>
-</segment>
-<segment>
-<pinref part="U5" gate="G$1" pin="TXD"/>
-<wire x1="403.86" y1="50.8" x2="408.94" y2="50.8" width="0.1524" layer="91"/>
-<label x="408.94" y="50.8" size="1.27" layer="95" xref="yes"/>
 </segment>
 </net>
@@
 <segment>
 <wire x1="236.22" y1="147.32" x2="233.68" y2="147.32" width="0.1524" layer="91"/>
-<wire x1="233.68" y1="147.32" x2="226.06" y2="147.32" width="0.1524" layer="91"/>
-<wire x1="226.06" y1="147.32" x2="226.06" y2="152.4" width="0.1524" layer="91"/>
+<wire x1="233.68" y1="147.32" x2="218.44" y2="147.32" width="0.1524" layer="91"/>
+<wire x1="218.44" y1="147.32" x2="218.44" y2="167.64" width="0.1524" layer="91"/>
 <pinref part="C5" gate="G$1" pin="1"/>
 <pinref part="ANT1" gate="ANT1" pin="RF_FEED"/>
@@
 <label x="17.78" y="119.38" size="1.27" layer="95" xref="yes"/>
 </segment>
-<segment>
-<pinref part="U5" gate="G$1" pin="CTS"/>
-<wire x1="403.86" y1="43.18" x2="408.94" y2="43.18" width="0.1524" layer="91"/>
-<label x="408.94" y="43.18" size="1.27" layer="95" xref="yes"/>
-</segment>
-</net>
+</net>
